File: hardware/humidity.kicad_pcb (KiCad board)
At the start: 2 copper layers, 15 x 25 mm, 24 parts, among them P101 CON-SENSOR2, P102 DEBUG, P103 BOOT, U101 XMC1XXX24, U102 HDC1080, U103 DRILL, U104 DRILL, U105 DRILL, U106 DRILL

Commit message: Add 3d information (tbc)
Parts:
- P101: footprint CON-SENSOR2 -> kicad-libraries:CON-SENSOR2
- RP101: footprint 4X0402 -> kicad-libraries:4X0402

Commit message: Add 3d information (final)
Parts:
- P101: footprint kicad-libraries:CON-SENSOR2 -> CON-SENSOR2
- RP101: footprint kicad-libraries:4X0402 -> 4X0402
- U102: footprint kicad-libraries:DFN6-30x30 -> kicad-libraries:DFN6-30x30_humidity
Connections:
- P101 pad 1: (no net) -> +5V
- RP102 pad 6: (no net) -> Net-(RP102-Pad6)
- RP102 pad 8: (no net) -> Net-(RP102-Pad8)
- U101 pad 11: (no net) -> Net-(U101-Pad11)
- U101 pad 12: (no net) -> Net-(U101-Pad12)
- U101 pad 13: (no net) -> Net-(U101-Pad13)
- U101 pad 14: (no net) -> Net-(U101-Pad14)
- U101 pad 16: (no net) -> Net-(U101-Pad16)
- U101 pad 18: (no net) -> Net-(U101-Pad18)
- U101 pad 2: (no net) -> Net-(U101-Pad2)
- U101 pad 20: (no net) -> Net-(U101-Pad20)
- U101 pad 21: (no net) -> Net-(U101-Pad21)
- U101 pad 3: (no net) -> Net-(U101-Pad3)
- U101 pad 5: (no net) -> Net-(U101-Pad5)
- U101 pad 6: (no net) -> Net-(U101-Pad6)
- U101 pad 8: (no net) -> Net-(U101-Pad8)
- U102 pad 3: (no net) -> Net-(U102-Pad3)
- U102 pad 4: (no net) -> Net-(U102-Pad4)

Commit message: define filter circuit
Parts:
- C102: value TBD -> 220pF
- RP101: value TBD -> 82
Connections:
- P101 pad 1: +5V -> (no net)
- RP102 pad 6: Net-(RP102-Pad6) -> (no net)
- RP102 pad 8: Net-(RP102-Pad8) -> (no net)
- U101 pad 11: Net-(U101-Pad11) -> (no net)
- U101 pad 12: Net-(U101-Pad12) -> (no net)
- U101 pad 13: Net-(U101-Pad13) -> (no net)
- U101 pad 14: Net-(U101-Pad14) -> (no net)
- U101 pad 16: Net-(U101-Pad16) -> (no net)
- U101 pad 18: Net-(U101-Pad18) -> (no net)
- U101 pad 2: Net-(U101-Pad2) -> (no net)
- U101 pad 20: Net-(U101-Pad20) -> (no net)
- U101 pad 21: Net-(U101-Pad21) -> (no net)
- U101 pad 3: Net-(U101-Pad3) -> (no net)
- U101 pad 5: Net-(U101-Pad5) -> (no net)
- U101 pad 6: Net-(U101-Pad6) -> (no net)
- U101 pad 8: Net-(U101-Pad8) -> (no net)
- U102 pad 3: Net-(U102-Pad3) -> (no net)
- U102 pad 4: Net-(U102-Pad4) -> (no net)
Changed lines of the file:
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@@
-(kicad_pcb (version 4) (host pcbnew 4.0.2+dfsg1-stable)
+(kicad_pcb (version 4) (host pcbnew 4.0.7-e0-6372~58~ubuntu16.10.1)
   (general
     (links 45)
@@
     (zones 0)
     (modules 24)
-    (nets 35)
+    (nets 17)
   )
   (page A4)
@@
     (pad_to_mask_clearance 0)
     (aux_axis_origin 0 0)
-    (visible_elements FFFF7F5F)
+    (visible_elements FFFF7F7F)
     (pcbplotparams
       (layerselection 0x00010_00000000)
@@
   (net 15 "Net-(P102-Pad1)")
   (net 16 "Net-(P103-Pad2)")
-  (net 17 +5V)
-  (net 18 "Net-(RP102-Pad6)")
-  (net 19 "Net-(RP102-Pad8)")
-  (net 20 "Net-(U101-Pad2)")
-  (net 21 "Net-(U101-Pad3)")
-  (net 22 "Net-(U101-Pad5)")
-  (net 23 "Net-(U101-Pad6)")
-  (net 24 "Net-(U101-Pad8)")
-  (net 25 "Net-(U101-Pad11)")
-  (net 26 "Net-(U101-Pad12)")
-  (net 27 "Net-(U101-Pad13)")
-  (net 28 "Net-(U101-Pad14)")
-  (net 29 "Net-(U101-Pad16)")
-  (net 30 "Net-(U101-Pad18)")
-  (net 31 "Net-(U101-Pad20)")
-  (net 32 "Net-(U101-Pad21)")
-  (net 33 "Net-(U102-Pad3)")
-  (net 34 "Net-(U102-Pad4)")
   (net_class Default "This is the default net class."
     (clearance 0.15)
@@
     (uvia_dia 0.3)
     (uvia_drill 0.1)
-    (add_net +5V)
     (add_net GND)
     (add_net "Net-(C102-Pad2)")
@@
     (add_net "Net-(P103-Pad2)")
     (add_net "Net-(R101-Pad1)")
-    (add_net "Net-(RP102-Pad6)")
-    (add_net "Net-(RP102-Pad8)")
-    (add_net "Net-(U101-Pad11)")
-    (add_net "Net-(U101-Pad12)")
-    (add_net "Net-(U101-Pad13)")
-    (add_net "Net-(U101-Pad14)")
-    (add_net "Net-(U101-Pad16)")
-    (add_net "Net-(U101-Pad18)")
-    (add_net "Net-(U101-Pad2)")
-    (add_net "Net-(U101-Pad20)")
-    (add_net "Net-(U101-Pad21)")
-    (add_net "Net-(U101-Pad3)")
-    (add_net "Net-(U101-Pad5)")
-    (add_net "Net-(U101-Pad6)")
-    (add_net "Net-(U101-Pad8)")
-    (add_net "Net-(U102-Pad3)")
-    (add_net "Net-(U102-Pad4)")
     (add_net S-CLK)
     (add_net S-CS)
@@
     (pad 5 smd rect (at -1.19888 0.8509) (size 0.44958 0.89916) (layers F.Cu F.Paste F.Mask)
       (net 9 SDA))
-    (pad 6 smd rect (at -0.39878 0.8509) (size 0.44958 0.89916) (layers F.Cu F.Paste F.Mask)
-      (net 18 "Net-(RP102-Pad6)"))
+    (pad 6 smd rect (at -0.39878 0.8509) (size 0.44958 0.89916) (layers F.Cu F.Paste F.Mask))
     (pad 7 smd rect (at 0.39878 0.8509) (size 0.44958 0.89916) (layers F.Cu F.Paste F.Mask)
       (net 10 SCL))
-    (pad 8 smd rect (at 1.19888 0.8509) (size 0.44958 0.89916) (layers F.Cu F.Paste F.Mask)
-      (net 19 "Net-(RP102-Pad8)"))
+    (pad 8 smd rect (at 1.19888 0.8509) (size 0.44958 0.89916) (layers F.Cu F.Paste F.Mask))
     (model Resistors_SMD/R_4x0603.wrl
       (at (xyz 0 0 0))
@@
       (effects (font (size 0.2 0.2) (thickness 0.05)))
     )
-    (fp_text value TBD (at 0 -0.275 270) (layer F.Fab)
+    (fp_text value 220pF (at 0 -0.275 270) (layer F.Fab)
       (effects (font (size 0.2 0.2) (thickness 0.05)))
     )
@@
     (pad 1 smd oval (at -2.025 -1.25 225) (size 1 0.3) (layers F.Cu F.Paste F.Mask)
       (net 11 S-MISO))
-    (pad 2 smd oval (at -2.025 -0.75 225) (size 1 0.3) (layers F.Cu F.Paste F.Mask)
-      (net 20 "Net-(U101-Pad2)"))
-    (pad 3 smd oval (at -2.025 -0.25 225) (size 1 0.3) (layers F.Cu F.Paste F.Mask)
-      (net 21 "Net-(U101-Pad3)"))
+    (pad 2 smd oval (at -2.025 -0.75 225) (size 1 0.3) (layers F.Cu F.Paste F.Mask))
+    (pad 3 smd oval (at -2.025 -0.25 225) (size 1 0.3) (layers F.Cu F.Paste F.Mask))
     (pad 4 smd oval (at -2.025 0.25 225) (size 1 0.3) (layers F.Cu F.Paste F.Mask)
       (net 16 "Net-(P103-Pad2)"))
-    (pad 5 smd oval (at -2.025 0.75 225) (size 1 0.3) (layers F.Cu F.Paste F.Mask)
-      (net 22 "Net-(U101-Pad5)"))
-    (pad 6 smd oval (at -2.025 1.25 225) (size 1 0.3) (layers F.Cu F.Paste F.Mask)
-      (net 23 "Net-(U101-Pad6)"))
+    (pad 5 smd oval (at -2.025 0.75 225) (size 1 0.3) (layers F.Cu F.Paste F.Mask))
+    (pad 6 smd oval (at -2.025 1.25 225) (size 1 0.3) (layers F.Cu F.Paste F.Mask))
     (pad 7 smd oval (at -1.25 2.025 315) (size 1 0.3) (layers F.Cu F.Paste F.Mask)
       (net 8 "Net-(R101-Pad1)"))
-    (pad 8 smd oval (at -0.75 2.025 315) (size 1 0.3) (layers F.Cu F.Paste F.Mask)
-      (net 24 "Net-(U101-Pad8)"))
+    (pad 8 smd oval (at -0.75 2.025 315) (size 1 0.3) (layers F.Cu F.Paste F.Mask))
     (pad 9 smd oval (at -0.25 2.025 315) (size 1 0.3) (layers F.Cu F.Paste F.Mask)
       (net 1 GND))
     (pad 10 smd oval (at 0.25 2.025 315) (size 1 0.3) (layers F.Cu F.Paste F.Mask)
       (net 2 VCC))
-    (pad 11 smd oval (at 0.75 2.025 315) (size 1 0.3) (layers F.Cu F.Paste F.Mask)
-      (net 25 "Net-(U101-Pad11)"))
-    (pad 12 smd oval (at 1.25 2.025 315) (size 1 0.3) (layers F.Cu F.Paste F.Mask)
-      (net 26 "Net-(U101-Pad12)"))
-    (pad 13 smd oval (at 2.025 1.25 225) (size 1 0.3) (layers F.Cu F.Paste F.Mask)
-      (net 27 "Net-(U101-Pad13)"))
-    (pad 14 smd oval (at 2.025 0.75 225) (size 1 0.3) (layers F.Cu F.Paste F.Mask)
-      (net 28 "Net-(U101-Pad14)"))
+    (pad 11 smd oval (at 0.75 2.025 315) (size 1 0.3) (layers F.Cu F.Paste F.Mask))
+    (pad 12 smd oval (at 1.25 2.025 315) (size 1 0.3) (layers F.Cu F.Paste F.Mask))
+    (pad 13 smd oval (at 2.025 1.25 225) (size 1 0.3) (layers F.Cu F.Paste F.Mask))
+    (pad 14 smd oval (at 2.025 0.75 225) (size 1 0.3) (layers F.Cu F.Paste F.Mask))
     (pad 15 smd oval (at 2.025 0.25 225) (size 1 0.3) (layers F.Cu F.Paste F.Mask)
       (net 15 "Net-(P102-Pad1)"))
-    (pad 16 smd oval (at 2.025 -0.25 225) (size 1 0.3) (layers F.Cu F.Paste F.Mask)
-      (net 29 "Net-(U101-Pad16)"))
+    (pad 16 smd oval (at 2.025 -0.25 225) (size 1 0.3) (layers F.Cu F.Paste F.Mask))
     (pad 17 smd oval (at 2.025 -0.75 225) (size 1 0.3) (layers F.Cu F.Paste F.Mask)
       (net 9 SDA))
-    (pad 18 smd oval (at 2.025 -1.25 225) (size 1 0.3) (layers F.Cu F.Paste F.Mask)
-      (net 30 "Net-(U101-Pad18)"))
+    (pad 18 smd oval (at 2.025 -1.25 225) (size 1 0.3) (layers F.Cu F.Paste F.Mask))
     (pad 19 smd oval (at 1.25 -2.025 315) (size 1 0.3) (layers F.Cu F.Paste F.Mask)
       (net 10 SCL))
-    (pad 20 smd oval (at 0.75 -2.025 315) (size 1 0.3) (layers F.Cu F.Paste F.Mask)
-      (net 31 "Net-(U101-Pad20)"))
-    (pad 21 smd oval (at 0.25 -2.025 315) (size 1 0.3) (layers F.Cu F.Paste F.Mask)
-      (net 32 "Net-(U101-Pad21)"))
+    (pad 20 smd oval (at 0.75 -2.025 315) (size 1 0.3) (layers F.Cu F.Paste F.Mask))
+    (pad 21 smd oval (at 0.25 -2.025 315) (size 1 0.3) (layers F.Cu F.Paste F.Mask))
     (pad 22 smd oval (at -0.25 -2.025 315) (size 1 0.3) (layers F.Cu F.Paste F.Mask)
       (net 12 S-CS))
@@
     (fp_line (start 6 -4.3) (end -6 -4.3) (layer F.Fab) (width 0.05))
     (fp_line (start -6 -4.3) (end -6 -0.25) (layer F.Fab) (width 0.05))
-    (pad 1 smd rect (at -3.75 -4.6 90) (size 0.6 1.8) (layers F.Cu F.Paste F.Mask)
-      (net 17 +5V))
+    (pad 1 smd rect (at -3.75 -4.6 90) (size 0.6 1.8) (layers F.Cu F.Paste F.Mask))
     (pad 2 smd rect (at -2.5 -4.6 90) (size 0.6 1.8) (layers F.Cu F.Paste F.Mask)
       (net 1 GND))
@@
       (effects (font (size 0.2 0.2) (thickness 0.05)))
     )
-    (fp_text value TBD (at -0.025 -0.45 90) (layer F.Fab)
+    (fp_text value 82 (at -0.025 -0.45 90) (layer F.Fab)
       (effects (font (size 0.2 0.2) (thickness 0.05)))
     )
@@
     (pad 2 smd rect (at 0 -1.55 90) (size 0.4 0.9) (layers F.Cu F.Paste F.Mask)
       (net 1 GND))
-    (pad 3 smd rect (at -0.95 -1.55 90) (size 0.4 0.9) (layers F.Cu F.Paste F.Mask)
-      (net 33 "Net-(U102-Pad3)"))
-    (pad 4 smd rect (at -0.95 1.55 90) (size 0.4 0.9) (layers F.Cu F.Paste F.Mask)
-      (net 34 "Net-(U102-Pad4)"))
+    (pad 3 smd rect (at -0.95 -1.55 90) (size 0.4 0.9) (layers F.Cu F.Paste F.Mask))
+    (pad 4 smd rect (at -0.95 1.55 90) (size 0.4 0.9) (layers F.Cu F.Paste F.Mask))
     (pad 5 smd rect (at 0 1.55 90) (size 0.4 0.9) (layers F.Cu F.Paste F.Mask)
       (net 2 VCC))

Commit message: specify processor
Parts:
- U101: value XMC1XXX24 -> XMC1100-16
Changed lines of the file:
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@@
-(kicad_pcb (version 4) (host pcbnew 4.0.7-e0-6372~58~ubuntu16.10.1)
+(kicad_pcb (version 4) (host pcbnew 4.0.7-e2-6376~58~ubuntu17.04.1)
   (general
     (links 45)
     (no_connects 0)
-    (area 139.909499 128.309499 155.290501 153.690501)
+    (area 139.244999 127.644999 275.49286 158.115)
     (thickness 1.6)
     (drawings 13)
@@
       (effects (font (size 0.3 0.3) (thickness 0.075)))
     )
-    (fp_text value XMC1XXX24 (at 0 0.8 225) (layer F.Fab)
+    (fp_text value XMC1100-16 (at 0 0.8 225) (layer F.Fab)
       (effects (font (size 0.3 0.3) (thickness 0.075)))
     )
