File: hardware/humidity-v2.kicad_pcb (KiCad board)
At the start: 2 copper layers, 15 x 25 mm, 24 parts, among them P101 CON-SENSOR2, P102 DEBUG, P103 BOOT, U101 XMC1100-16, U102 HDC1080, U103 DRILL, U104 DRILL, U105 DRILL, U106 DRILL

Commit message: fix coordinate origin
Parts:
- moved VAL 0.30 mm to (147.6, 147.0)
- moved G*** 0.20 mm to (147.6, 135.5)
Changed lines of the file:
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@@
-(kicad_pcb (version 4) (host pcbnew 4.0.7-e2-6376~58~ubuntu17.04.1)
+(kicad_pcb (version 4) (host pcbnew 4.0.7-e2-6376~61~ubuntu18.04.1)
   (general
     (links 45)
@@
     (pad_drill 0.6)
     (pad_to_mask_clearance 0)
-    (aux_axis_origin 0 0)
-    (visible_elements FFFF7F7F)
+    (aux_axis_origin 140.1 128.5)
+    (grid_origin 140.1 128.5)
+    (visible_elements FFFFBF7F)
     (pcbplotparams
       (layerselection 0x00010_00000000)
@@
   )
   (module kicad-libraries:WEEE_7mm (layer B.Cu)
-    (at 147.6 135.3 270)
+    (at 147.6 135.5 270)
     (fp_text reference G*** (at 0 0 270) (layer B.SilkS) hide
       (effects (font (thickness 0.3)) (justify mirror))
@@
   )
   (module kicad-libraries:CE_5mm (layer B.Cu)
-    (at 147.6 146.7 270)
+    (at 147.6 147 270)
     (fp_text reference VAL (at 0 0 270) (layer B.SilkS) hide
       (effects (font (size 1.143 1.143) (thickness 0.1778)) (justify mirror))

Commit message: Change capacitor footprint(s) to C0402F
Parts:
- C101: footprint C0805 -> kicad-libraries:C0805
- C102: footprint C0402E -> kicad-libraries:C0402F
- C103, C104, C105: footprint C0603F -> kicad-libraries:C0603F
- D101: footprint D0603E -> kicad-libraries:D0603F
- P101: footprint CON-SENSOR2 -> kicad-libraries:CON-SENSOR2
- R101: footprint R0603F -> kicad-libraries:R0603F
- RP101: footprint 4X0402 -> kicad-libraries:4X0402
- RP102: footprint 0603X4 -> kicad-libraries:0603X4
- U103, U104, U105, U106: footprint DRILL_NP -> kicad-libraries:DRILL_NP
Connections:
- P101 pad 1: (no net) -> +5V
- RP102 pad 6: (no net) -> Net-(RP102-Pad6)
- RP102 pad 8: (no net) -> Net-(RP102-Pad8)
- U101 pad 11: (no net) -> Net-(U101-Pad11)
- U101 pad 12: (no net) -> Net-(U101-Pad12)
- U101 pad 13: (no net) -> Net-(U101-Pad13)
- U101 pad 14: (no net) -> Net-(U101-Pad14)
- U101 pad 16: (no net) -> Net-(U101-Pad16)
- U101 pad 18: (no net) -> Net-(U101-Pad18)
- U101 pad 2: (no net) -> Net-(U101-Pad2)
- U101 pad 20: (no net) -> Net-(U101-Pad20)
- U101 pad 21: (no net) -> Net-(U101-Pad21)
- U101 pad 3: (no net) -> Net-(U101-Pad3)
- U101 pad 5: (no net) -> Net-(U101-Pad5)
- U101 pad 6: (no net) -> Net-(U101-Pad6)
- U101 pad 8: (no net) -> Net-(U101-Pad8)
- U102 pad 3: (no net) -> Net-(U102-Pad3)
- U102 pad 4: (no net) -> Net-(U102-Pad4)

Commit message: Fix "Status" marking
Other:
- board text added: "Status"
- board text removed: "status"
Changed lines of the file:
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@@
     (effects (font (size 0.7 0.7) (thickness 0.15)))
   )
-  (gr_text status (at 147.6 129.5) (layer F.SilkS)
+  (gr_text Status (at 147.6 129.5) (layer F.SilkS)
     (effects (font (size 0.7 0.7) (thickness 0.15)))
   )
