File: hardware/humidity-v2.kicad_pcb (KiCad board)
At the start: 2 copper layers, 15 x 25 mm, 24 parts, among them P101 CON-SENSOR2, P102 DEBUG, P103 BOOT, U101 XMC1100-16, U102 HDC1080, U103 DRILL, U104 DRILL, U105 DRILL, U106 DRILL

Commit message: Data Cleanup
Parts:
- moved U104 64.4 mm to (151.7, 86.6), turned to 90 degrees
- moved Fiducial_Mark 60.6 mm to (152.7, 91.6), turned to 90 degrees
- moved P101 58.5 mm to (141.7, 84.1), turned to 180 degrees
- moved G*** 57.2 mm to (151.5, 93.9), turned to 180 degrees
- moved VAL 55.4 mm to (147.7, 91.6), turned to 0 degrees
- moved U106 55.2 mm to (151.7, 96.6), turned to 90 degrees
- moved Fiducial_Mark 54.1 mm to (138.2, 85.6), turned to 90 degrees
- moved C105 54.1 mm to (146.8, 92.0), turned to 90 degrees
- moved C101 52.9 mm to (144.1, 90.7), turned to 180 degrees
- moved C103 51.1 mm to (143.9, 92.2), turned to 180 degrees
- moved U102 50.4 mm to (146.8, 95.8), turned to 180 degrees
- moved G*** 49.8 mm to (141.7, 91.6), turned to 0 degrees
- moved U103 49.1 mm to (131.7, 86.6), turned to 90 degrees
- moved RP101 48.8 mm to (139.8, 91.0), turned to 180 degrees
- moved C102 47.5 mm to (137.3, 90.5), turned to 0 degrees
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Routing:
- net VCC: track 33.1 -> 41.8 mm
Other:
- board size 15 x 25 mm -> 25 x 15 mm
- net class Default removed
- board text added: "Copyright Tinkerforge GmbH 2023. This documentation describes Open Hardware and is licensed under the CERN OHL v. 1.1. You may redistribute and modify this documentation under the terms of the CERN OHL v.1.1. (http://ohwr.org/cernohl). This documentation is distributed WITHOUT ANY EXPRESS OR IMPLIED WARRANTY, INCLUDING OF MERCHANTABILITY, SATISFACTORY QUALITY AND FITNESS FOR A PARTICULAR PURPOSE.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"
- board text removed: "Copyright Tinkerforge GmbH 2017. This documentation describes Open Hardware and is licensed under the CERN OHL v. 1.1. You may redistribute and modify this documentation under the terms of the CERN OHL v.1.1. (http://ohwr.org/cernohl). This documentation is distributed WITHOUT ANY EXPRESS OR IMPLIED WARRANTY, INCLUDING OF MERCHANTABILITY, SATISFACTORY QUALITY AND FITNESS FOR A PARTICULAR PURPOSE.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"
